File: NodeLoRaGroveKitty.kicad_pcb (KiCad board)
At the start: 2 copper layers, 50 x 50 mm, 42 parts, among them IC1 CP2104, J1 10118192-0001LF, P2 Battery, P4 A0, P5 D9, P6 I2C, Q1 MMBT2222A, Q2 MMBT2222A, U1 AP2114, U2 MCP73831T-2ATI/OT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

Commit message: Fix gnd
Routing:
- net GND: track 112.3 -> 153.0 mm, vias 16 -> 34
- net (no net): track 15.5 -> 6.72 mm, vias 3 -> 1
Changed lines of the file:
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@@
     (thickness 1.6)
     (drawings 16)
-    (tracks 616)
+    (tracks 660)
     (zones 0)
     (modules 42)
@@
     (arrow2b (pts (xy 120.16 82.64) (xy 120.746421 83.766504)))
   )
-  (segment (start 132.86 87.56) (end 132.86 86.6) (width 0.3) (layer F.Cu) (net 0))
-  (segment (start 132.86 86.6) (end 133.18 86.28) (width 0.3) (layer F.Cu) (net 0))
-  (via (at 133.18 86.28) (size 0.7) (drill 0.5) (layers F.Cu B.Cu) (net 0))
-  (segment (start 126.81 88.84) (end 131.58 88.84) (width 0.3) (layer B.Cu) (net 0))
-  (via (at 132.86 87.56) (size 0.7) (drill 0.5) (layers F.Cu B.Cu) (net 0))
-  (segment (start 131.58 88.84) (end 132.86 87.56) (width 0.3) (layer B.Cu) (net 0))
-  (segment (start 126.81 88.84) (end 127.56 88.84) (width 0.3) (layer B.Cu) (net 0))
-  (segment (start 126.82 88.85) (end 126.81 88.84) (width 0.3) (layer F.Cu) (net 0))
   (segment (start 157.56 119.98) (end 158.64 118.9) (width 0.3) (layer F.Cu) (net 0))
   (via (at 158.64 113.71) (size 0.7) (drill 0.5) (layers F.Cu B.Cu) (net 0))
   (segment (start 158.64 118.9) (end 158.64 113.71) (width 0.3) (layer F.Cu) (net 0))
+  (segment (start 142.6 84) (end 141.4 84) (width 0.3) (layer F.Cu) (net 1))
+  (via (at 141.4 84) (size 0.7) (drill 0.5) (layers F.Cu B.Cu) (net 1))
+  (segment (start 144.6 84.8) (end 143.8 84) (width 0.3) (layer B.Cu) (net 1))
+  (segment (start 143.8 84) (end 142.6 84) (width 0.3) (layer B.Cu) (net 1))
+  (via (at 142.6 84) (size 0.7) (drill 0.5) (layers F.Cu B.Cu) (net 1))
+  (segment (start 145.2 86.2) (end 145.2 85.4) (width 0.3) (layer F.Cu) (net 1))
+  (segment (start 145.2 85.4) (end 144.6 84.8) (width 0.3) (layer F.Cu) (net 1))
+  (via (at 144.6 84.8) (size 0.7) (drill 0.5) (layers F.Cu B.Cu) (net 1))
+  (segment (start 145.17 87.87) (end 145.17 86.23) (width 0.3) (layer B.Cu) (net 1))
+  (segment (start 145.17 86.23) (end 145.2 86.2) (width 0.3) (layer B.Cu) (net 1))
+  (via (at 145.2 86.2) (size 0.7) (drill 0.5) (layers F.Cu B.Cu) (net 1))
+  (segment (start 141.4 86.2) (end 140.2 86.2) (width 0.3) (layer B.Cu) (net 1))
+  (via (at 140.2 86.2) (size 0.7) (drill 0.5) (layers F.Cu B.Cu) (net 1))
+  (segment (start 142.6 86.2) (end 141.4 86.2) (width 0.3) (layer F.Cu) (net 1))
+  (via (at 141.4 86.2) (size 0.7) (drill 0.5) (layers F.Cu B.Cu) (net 1))
+  (segment (start 142.63 87.87) (end 142.63 86.23) (width 0.3) (layer B.Cu) (net 1))
+  (segment (start 142.63 86.23) (end 142.6 86.2) (width 0.3) (layer B.Cu) (net 1))
+  (via (at 142.6 86.2) (size 0.7) (drill 0.5) (layers F.Cu B.Cu) (net 1))
+  (segment (start 142.63 87.87) (end 142.63 86.63) (width 0.3) (layer B.Cu) (net 1))
+  (segment (start 142.63 86.63) (end 142.4 86.4) (width 0.3) (layer B.Cu) (net 1))
+  (segment (start 132.8 84.2) (end 134.4 84.2) (width 0.3) (layer B.Cu) (net 1))
+  (via (at 134.4 84.2) (size 0.7) (drill 0.5) (layers F.Cu B.Cu) (net 1))
+  (segment (start 131.2 84.6) (end 132.4 84.6) (width 0.3) (layer F.Cu) (net 1))
+  (segment (start 132.4 84.6) (end 132.8 84.2) (width 0.3) (layer F.Cu) (net 1))
+  (via (at 132.8 84.2) (size 0.7) (drill 0.5) (layers F.Cu B.Cu) (net 1))
+  (segment (start 130.53 86.16) (end 130.53 85.27) (width 0.3) (layer B.Cu) (net 1))
+  (segment (start 130.53 85.27) (end 131.2 84.6) (width 0.3) (layer B.Cu) (net 1))
+  (via (at 131.2 84.6) (size 0.7) (drill 0.5) (layers F.Cu B.Cu) (net 1))
+  (segment (start 128 86.8) (end 129.2 86.8) (width 0.3) (layer F.Cu) (net 1))
+  (via (at 129.2 86.8) (size 0.7) (drill 0.5) (layers F.Cu B.Cu) (net 1))
+  (segment (start 126.8 89.2) (end 128 89.2) (width 0.3) (layer B.Cu) (net 1))
+  (via (at 128 89.2) (size 0.7) (drill 0.5) (layers F.Cu B.Cu) (net 1))
+  (segment (start 125.4 89.2) (end 126.8 89.2) (width 0.3) (layer F.Cu) (net 1))
+  (via (at 126.8 89.2) (size 0.7) (drill 0.5) (layers F.Cu B.Cu) (net 1))
+  (segment (start 125.93 90.33) (end 125.4 89.8) (width 0.3) (layer B.Cu) (net 1))
+  (segment (start 125.4 89.8) (end 125.4 89.2) (width 0.3) (layer B.Cu) (net 1))
+  (via (at 125.4 89.2) (size 0.7) (drill 0.5) (layers F.Cu B.Cu) (net 1))
+  (segment (start 126.82 90.33) (end 125.93 90.33) (width 0.3) (layer B.Cu) (net 1))
+  (segment (start 126.8 86.8) (end 125.4 86.8) (width 0.3) (layer F.Cu) (net 1))
+  (via (at 125.4 86.8) (size 0.7) (drill 0.5) (layers F.Cu B.Cu) (net 1))
+  (segment (start 128 86.8) (end 126.8 86.8) (width 0.3) (layer B.Cu) (net 1))
+  (via (at 126.8 86.8) (size 0.7) (drill 0.5) (layers F.Cu B.Cu) (net 1))
+  (segment (start 124.4 85.25) (end 125.012 85.25) (width 0.3) (layer F.Cu) (net 1))
+  (segment (start 123.742 85.25) (end 124.4 85.25) (width 0.3) (layer F.Cu) (net 1))
+  (segment (start 124.4 85.25) (end 126.45 85.25) (width 0.3) (layer F.Cu) (net 1))
+  (segment (start 126.45 85.25) (end 128 86.8) (width 0.3) (layer F.Cu) (net 1))
+  (via (at 128 86.8) (size 0.7) (drill 0.5) (layers F.Cu B.Cu) (net 1))
+  (segment (start 133 88.6) (end 133 87.4) (width 0.3) (layer B.Cu) (net 1))
+  (segment (start 133 87.4) (end 133 86.4) (width 0.3) (layer B.Cu) (net 1))
+  (segment (start 133 86.4) (end 133 87.4) (width 0.3) (layer F.Cu) (net 1))
+  (via (at 133 87.4) (size 0.7) (drill 0.5) (layers F.Cu B.Cu) (net 1))
+  (via (at 133 86.4) (size 0.7) (drill 0.5) (layers F.Cu B.Cu) (net 1))
+  (segment (start 131.27 90.33) (end 133 88.6) (width 0.3) (layer B.Cu) (net 1))
+  (segment (start 126.82 90.33) (end 131.27 90.33) (width 0.3) (layer B.Cu) (net 1))
   (segment (start 167.21 100.97) (end 165.8 100.97) (width 0.3) (layer F.Cu) (net 1))
   (segment (start 165.8 100.97) (end 165.03 101.74) (width 0.3) (layer F.Cu) (net 1))
@@
   (via (at 159.26 87.54) (size 0.7) (drill 0.5) (layers F.Cu B.Cu) (net 1))
   (via (at 162.53 85.19) (size 0.7) (drill 0.5) (layers F.Cu B.Cu) (net 1))
-  (segment (start 123.742 85.25) (end 125.012 85.25) (width 0.3) (layer F.Cu) (net 1))
   (segment (start 123.742 90.33) (end 126.82 90.33) (width 0.3) (layer F.Cu) (net 1))
-  (via (at 126.82 90.33) (size 0.7) (drill 0.5) (layers F.Cu B.Cu) (net 1))
   (segment (start 164.76 97.84) (end 164.76 102.14) (width 0.3) (layer F.Cu) (net 1))
   (segment (start 164.76 102.14) (end 164.26 102.64) (width 0.3) (layer F.Cu) (net 1))

Commit message: checksum
Routing:
- net GND: track 153.0 -> 136.4 mm, vias 34 -> 31
- net (no net): track 6.72 -> 4.78 mm, vias 1 -> 3
Changed lines of the file:
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@@
-(kicad_pcb (version 4) (host pcbnew 4.0.5)
+(kicad_pcb (version 4) (host pcbnew 4.0.6)
   (general
     (links 110)
-    (no_connects 0)
-    (area 120.109999 82.589999 170.210001 132.690001)
+    (no_connects 1)
+    (area 110.748899 74.664999 170.748875 139.97)
     (thickness 1.6)
     (drawings 16)
-    (tracks 660)
+    (tracks 657)
     (zones 0)
     (modules 42)
@@
     (46 B.CrtYd user)
     (47 F.CrtYd user)
-    (48 B.Fab user)
-    (49 F.Fab user)
+    (48 B.Fab user hide)
+    (49 F.Fab user hide)
   )
   (setup
@@
     (arrow2b (pts (xy 120.16 82.64) (xy 120.746421 83.766504)))
   )
-  (segment (start 157.56 119.98) (end 158.64 118.9) (width 0.3) (layer F.Cu) (net 0))
-  (via (at 158.64 113.71) (size 0.7) (drill 0.5) (layers F.Cu B.Cu) (net 0))
-  (segment (start 158.64 118.9) (end 158.64 113.71) (width 0.3) (layer F.Cu) (net 0))
+  (segment (start 133 87.4) (end 133 86.4) (width 0.3) (layer B.Cu) (net 0))
+  (segment (start 133 86.4) (end 133 87.4) (width 0.3) (layer F.Cu) (net 0))
+  (via (at 133 87.4) (size 0.7) (drill 0.5) (layers F.Cu B.Cu) (net 0))
+  (via (at 133 86.4) (size 0.7) (drill 0.5) (layers F.Cu B.Cu) (net 0))
+  (segment (start 167.21 100.97) (end 165.8 100.97) (width 0.3) (layer F.Cu) (net 0))
+  (segment (start 165.84 100.97) (end 167.21 100.97) (width 0.3) (layer F.Cu) (net 0))
+  (via (at 167.21 100.97) (size 0.7) (drill 0.5) (layers F.Cu B.Cu) (net 0))
+  (segment (start 126.71 89.05) (end 127.89 89.05) (width 0.3) (layer B.Cu) (net 1))
+  (segment (start 127.89 89.05) (end 127.96 88.98) (width 0.3) (layer B.Cu) (net 1))
+  (via (at 127.96 88.98) (size 0.7) (drill 0.5) (layers F.Cu B.Cu) (net 1))
+  (segment (start 125.375877 89.100415) (end 126.659585 89.100415) (width 0.3) (layer F.Cu) (net 1))
+  (segment (start 126.659585 89.100415) (end 126.71 89.05) (width 0.3) (layer F.Cu) (net 1))
+  (via (at 126.71 89.05) (size 0.7) (drill 0.5) (layers F.Cu B.Cu) (net 1))
+  (segment (start 122.29 90.36) (end 123.56 90.36) (width 0.3) (layer B.Cu) (net 1))
+  (segment (start 123.56 90.36) (end 124.819585 89.100415) (width 0.3) (layer B.Cu) (net 1))
+  (segment (start 124.819585 89.100415) (end 125.375877 89.100415) (width 0.3) (layer B.Cu) (net 1))
+  (via (at 125.375877 89.100415) (size 0.7) (drill 0.5) (layers F.Cu B.Cu) (net 1))
+  (segment (start 132.46 89.14) (end 131.41 89.14) (width 0.3) (layer F.Cu) (net 1))
+  (segment (start 131.41 89.14) (end 131.16 88.89) (width 0.3) (layer F.Cu) (net 1))
+  (segment (start 131.16 88.89) (end 131.16 86.72) (width 0.3) (layer F.Cu) (net 1))
+  (segment (start 131.16 86.72) (end 130.72 86.28) (width 0.3) (layer F.Cu) (net 1))
+  (segment (start 130.72 86.28) (end 130.65 86.28) (width 0.3) (layer F.Cu) (net 1))
+  (segment (start 130.65 86.28) (end 130.53 86.16) (width 0.3) (layer F.Cu) (net 1))
+  (segment (start 165.03 101.74) (end 165.03 100.16) (width 0.3) (layer F.Cu) (net 1))
+  (segment (start 165.03 100.16) (end 164.91 100.04) (width 0.3) (layer F.Cu) (net 1))
   (segment (start 142.6 84) (end 141.4 84) (width 0.3) (layer F.Cu) (net 1))
   (via (at 141.4 84) (size 0.7) (drill 0.5) (layers F.Cu B.Cu) (net 1))
@@
   (segment (start 128 86.8) (end 129.2 86.8) (width 0.3) (layer F.Cu) (net 1))
   (via (at 129.2 86.8) (size 0.7) (drill 0.5) (layers F.Cu B.Cu) (net 1))
-  (segment (start 126.8 89.2) (end 128 89.2) (width 0.3) (layer B.Cu) (net 1))
-  (via (at 128 89.2) (size 0.7) (drill 0.5) (layers F.Cu B.Cu) (net 1))
-  (segment (start 125.4 89.2) (end 126.8 89.2) (width 0.3) (layer F.Cu) (net 1))
-  (via (at 126.8 89.2) (size 0.7) (drill 0.5) (layers F.Cu B.Cu) (net 1))
-  (segment (start 125.93 90.33) (end 125.4 89.8) (width 0.3) (layer B.Cu) (net 1))
-  (segment (start 125.4 89.8) (end 125.4 89.2) (width 0.3) (layer B.Cu) (net 1))
-  (via (at 125.4 89.2) (size 0.7) (drill 0.5) (layers F.Cu B.Cu) (net 1))
-  (segment (start 126.82 90.33) (end 125.93 90.33) (width 0.3) (layer B.Cu) (net 1))
   (segment (start 126.8 86.8) (end 125.4 86.8) (width 0.3) (layer F.Cu) (net 1))
   (via (at 125.4 86.8) (size 0.7) (drill 0.5) (layers F.Cu B.Cu) (net 1))
@@
   (segment (start 126.45 85.25) (end 128 86.8) (width 0.3) (layer F.Cu) (net 1))
   (via (at 128 86.8) (size 0.7) (drill 0.5) (layers F.Cu B.Cu) (net 1))
-  (segment (start 133 88.6) (end 133 87.4) (width 0.3) (layer B.Cu) (net 1))
-  (segment (start 133 87.4) (end 133 86.4) (width 0.3) (layer B.Cu) (net 1))
-  (segment (start 133 86.4) (end 133 87.4) (width 0.3) (layer F.Cu) (net 1))
-  (via (at 133 87.4) (size 0.7) (drill 0.5) (layers F.Cu B.Cu) (net 1))
-  (via (at 133 86.4) (size 0.7) (drill 0.5) (layers F.Cu B.Cu) (net 1))
-  (segment (start 131.27 90.33) (end 133 88.6) (width 0.3) (layer B.Cu) (net 1))
-  (segment (start 126.82 90.33) (end 131.27 90.33) (width 0.3) (layer B.Cu) (net 1))
-  (segment (start 167.21 100.97) (end 165.8 100.97) (width 0.3) (layer F.Cu) (net 1))
-  (segment (start 165.8 100.97) (end 165.03 101.74) (width 0.3) (layer F.Cu) (net 1))
   (via (at 165.03 101.74) (size 0.7) (drill 0.5) (layers F.Cu B.Cu) (net 1))
   (segment (start 156.86 95.439998) (end 156.86 98.3) (width 0.3) (layer F.Cu) (net 1))
@@
   (segment (start 144.925596 113.274404) (end 140.35 117.85) (width 0.3) (layer B.Cu) (net 1))
   (segment (start 154.05858 113.274404) (end 144.925596 113.274404) (width 0.3) (layer B.Cu) (net 1))
-  (segment (start 130.72 86.28) (end 130.65 86.28) (width 0.3) (layer F.Cu) (net 1))
-  (segment (start 130.65 86.28) (end 130.53 86.16) (width 0.3) (layer F.Cu) (net 1))
   (via (at 130.53 86.16) (size 0.7) (drill 0.5) (layers F.Cu B.Cu) (net 1))
   (segment (start 154.05858 89.144404) (end 155.12058 89.144404) (width 0.3) (layer B.Cu) (net 1))
@@
   (segment (start 157.03 124.01) (end 157.03 122.41) (width 0.3) (layer F.Cu) (net 1))
   (via (at 157.03 122.41) (size 0.7) (drill 0.5) (layers F.Cu B.Cu) (net 1))
-  (segment (start 131.16 86.72) (end 130.72 86.28) (width 0.3) (layer F.Cu) (net 1))
-  (segment (start 131.16 87.94) (end 131.16 86.72) (width 0.3) (layer F.Cu) (net 1))
-  (segment (start 132.36 89.14) (end 131.16 87.94) (width 0.3) (layer F.Cu) (net 1))
-  (segment (start 132.46 89.14) (end 132.36 89.14) (width 0.3) (layer F.Cu) (net 1))
-  (segment (start 164.91 100.04) (end 165.84 100.97) (width 0.3) (layer F.Cu) (net 1))
-  (segment (start 165.84 100.97) (end 167.21 100.97) (width 0.3) (layer F.Cu) (net 1))
-  (via (at 167.21 100.97) (size 0.7) (drill 0.5) (layers F.Cu B.Cu) (net 1))
   (segment (start 164.91 96.64) (end 164.91 100.04) (width 0.3) (layer F.Cu) (net 1))
   (segment (start 154.39 87.54) (end 154.05858 87.87142) (width 0.3) (layer B.Cu) (net 1))
@@
   (via (at 162.53 85.19) (size 0.7) (drill 0.5) (layers F.Cu B.Cu) (net 1))
   (segment (start 123.742 90.33) (end 126.82 90.33) (width 0.3) (layer F.Cu) (net 1))
-  (segment (start 164.76 97.84) (end 164.76 102.14) (width 0.3) (layer F.Cu) (net 1))
-  (segment (start 164.76 102.14) (end 164.26 102.64) (width 0.3) (layer F.Cu) (net 1))
   (segment (start 164.91 96.64) (end 164.91 97.69) (width 0.3) (layer F.Cu) (net 1))
   (segment (start 164.91 97.69) (end 164.76 97.84) (width 0.3) (layer F.Cu) (net 1))
@@
   (via (at 146.16 90.04) (size 0.7) (drill 0.5) (layers F.Cu B.Cu) (net 55))
   (segment (start 152.16 87.64) (end 146.76 87.64) (width 0.3) (layer F.Cu) (net 55))
-  (segment (start 162.41 93.94) (end 156.66 93.94) (width 0.3) (layer F.Cu) (net 56))
+  (segment (start 161.01 94.57) (end 161.01 94.39) (width 0.3) (layer F.Cu) (net 56))
+  (segment (start 161.01 104.29) (end 161.01 94.57) (width 0.3) (layer F.Cu) (net 56))
+  (segment (start 162.41 93.94) (end 161.04 93.94) (width 0.3) (layer F.Cu) (net 56))
+  (segment (start 161.04 93.94) (end 156.66 93.94) (width 0.3) (layer F.Cu) (net 56))
+  (segment (start 161.01 94.57) (end 161.01 93.97) (width 0.3) (layer F.Cu) (net 56))
+  (segment (start 161.01 93.97) (end 161.04 93.94) (width 0.3) (layer F.Cu) (net 56))
   (segment (start 156.66 93.94) (end 155.91 93.19) (width 0.3) (layer F.Cu) (net 56))
   (segment (start 155.91 93.19) (end 155.91 92.19) (width 0.3) (layer F.Cu) (net 56))
@@
   (segment (start 161.91 105.94) (end 161.91 105.19) (width 0.3) (layer F.Cu) (net 56))
   (segment (start 161.91 105.19) (end 161.01 104.29) (width 0.3) (layer F.Cu) (net 56))
-  (segment (start 161.01 104.29) (end 161.01 94.39) (width 0.3) (layer F.Cu) (net 56))
-  (segment (start 161.01 94.39) (end 161.46 93.94) (width 0.3) (layer F.Cu) (net 56))
   (segment (start 161.46 93.94) (end 162.41 93.94) (width 0.3) (layer F.Cu) (net 56))
   (segment (start 157.31 108.04) (end 157.31 109.34) (width 0.3) (layer F.Cu) (net 57))

Commit message: fix connects
Routing:
- net (no net): track 4.78 -> 2.00 mm
Changed lines of the file:
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@@
   (general
     (links 110)
-    (no_connects 1)
+    (no_connects 0)
     (area 110.748899 74.664999 170.748875 139.97)
     (thickness 1.6)
     (drawings 16)
-    (tracks 657)
+    (tracks 655)
     (zones 0)
     (modules 42)
@@
   (via (at 133 87.4) (size 0.7) (drill 0.5) (layers F.Cu B.Cu) (net 0))
   (via (at 133 86.4) (size 0.7) (drill 0.5) (layers F.Cu B.Cu) (net 0))
-  (segment (start 167.21 100.97) (end 165.8 100.97) (width 0.3) (layer F.Cu) (net 0))
-  (segment (start 165.84 100.97) (end 167.21 100.97) (width 0.3) (layer F.Cu) (net 0))
   (via (at 167.21 100.97) (size 0.7) (drill 0.5) (layers F.Cu B.Cu) (net 0))
   (segment (start 126.71 89.05) (end 127.89 89.05) (width 0.3) (layer B.Cu) (net 1))
